File: project/68000sbc.kicad_pcb (KiCad board)
At the start: 2 copper layers, 127 x 90.8 mm, 49 parts, among them J1 USB_B, J2 5V FTDI SERIAL, J3 RTC (SparkFun BOB-10160), J4 CFCARD/IDE, J5 EXPANSION (F.Cu), J6 EXPANSION (B.Cu), SW1 RESET, SW2 BTN1, U1 74HC139, U2 74HC14, U3 TMP68HC000P-12, U4 AS6C4008-55PCN, U5 28C256, U6 AS6C4008-55PCN, U7 28C256, U8 TL16C550, X1 12MHz, X2 12MHz

Commit message: Add local build and fabrication draft workflow
Connections:
- net /R,~W renamed /R,~{W}
- net /~A20 renamed /~{A20}
- net /~A22 renamed /~{A22}
- net /~AS renamed /~{AS}
- net /~BTN1 renamed /~{BTN1}
- net /~CFLED renamed /~{CFLED}
- net /~HALT renamed /~{HALT}
- net /~IRQ renamed /~{IRQ}
- net /~LDS renamed /~{LDS}
- net /~RDL renamed /~{RDL}
- net /~RDU renamed /~{RDU}
- net /~RESET renamed /~{RESET}
- net /~RESETBTN renamed /~{RESETBTN}
- net /~RTC_SS renamed /~{RTC_SS}
- net /~UDS renamed /~{UDS}
- net /~WRL renamed /~{WRL}
- net /~WRU renamed /~{WRU}
- J1 pad 1: Net-(J1-Pad1) -> unconnected-(J1-VBUS-Pad1)
- J1 pad 2: Net-(J1-Pad2) -> unconnected-(J1-D--Pad2)
- J1 pad 3: Net-(J1-Pad3) -> unconnected-(J1-D+-Pad3)
- J1 pad 5: GND -> (no net)
- J2 pad 2: Net-(J2-Pad2) -> unconnected-(J2-Pin_2-Pad2)
- J2 pad 3: Net-(J2-Pad3) -> unconnected-(J2-Pin_3-Pad3)
- J2 pad 6: Net-(J2-Pad6) -> unconnected-(J2-Pin_6-Pad6)
- J4 pad 20: Net-(J4-Pad20) -> unconnected-(J4-Pin_20-Pad20)
- J4 pad 21: Net-(J4-Pad21) -> unconnected-(J4-Pin_21-Pad21)
- J4 pad 27: Net-(J4-Pad27) -> unconnected-(J4-Pin_27-Pad27)
- J4 pad 28: Net-(J4-Pad28) -> unconnected-(J4-Pin_28-Pad28)
- J4 pad 29: Net-(J4-Pad29) -> unconnected-(J4-Pin_29-Pad29)
- J4 pad 32: Net-(J4-Pad32) -> unconnected-(J4-Pin_32-Pad32)
- J4 pad 34: Net-(J4-Pad34) -> unconnected-(J4-Pin_34-Pad34)
- J4 pad 44: Net-(J4-Pad44) -> unconnected-(J4-Pin_44-Pad44)
- JP1 pad 1: Net-(J2-Pad3) -> unconnected-(JP1-A-Pad1)
- JP1 pad 3: Net-(J1-Pad1) -> unconnected-(JP1-B-Pad3)
- R3 pad 1: Net-(C11-Pad1) -> Net-(R3-Pad1)
- U1 pad 10: Net-(U1-Pad10) -> unconnected-(U1B-O2-Pad10)
- U1 pad 6: Net-(U1-Pad6) -> unconnected-(U1A-O2-Pad6)
- U1 pad 7: Net-(U1-Pad7) -> unconnected-(U1A-O3-Pad7)
- U1 pad 9: Net-(U1-Pad9) -> unconnected-(U1B-O3-Pad9)
- U2 pad 5: Net-(C11-Pad1) -> Net-(R3-Pad1)
- U8 pad 17: Net-(U8-Pad17) -> unconnected-(U8-XOUT-Pad17)
- U8 pad 23: Net-(U8-Pad23) -> unconnected-(U8-DDIS-Pad23)
- U8 pad 24: Net-(U8-Pad24) -> unconnected-(U8-~{TXRDY}-Pad24)
- U8 pad 29: Net-(U8-Pad29) -> unconnected-(U8-~{RXRDY}-Pad29)
Routing:
- net (no net): track 0.00 -> 39.2 mm
- net Net-(J2-Pad3): track 25.8 -> 0.00 mm
- net Net-(J1-Pad1): track 13.5 -> 0.00 mm
Other:
- net class Default removed
- net class Thicc removed
- board text added: "68k MAGIC"
- board text added: "R/~{W}"
- board text added: "cartheur"
- board text added: "~{AS}"
- board text added: "~{BERR}"
- board text added: "~{BGACK}"
- board text added: "~{BG}"
- board text added: "~{BR}"
- board text added: "~{DTACK}"
- board text added: "~{DTACK} GROUNDED!!"
- board text added: "~{HALT}"
- board text added: "~{IPL0}"
- board text added: "~{IPL1}"
- board text added: "~{IPL2}"
- board text added: "~{LDS}"
- board text added: "~{RDL}"
- board text added: "~{RDU}"
- board text added: "~{RESET}"
- board text added: "~{RST}"
- board text added: "~{SS}"
- board text added: "~{UDS}"
- board text added: "~{VMA}"
- board text added: "~{VPA}"
- board text added: "~{WRL}"
- board text added: "~{WRU}"
- board text removed: "68k nano"
- board text removed: "R/~W"
- board text removed: "single board computer"
- board text removed: "~AS"
- board text removed: "~BERR"
- board text removed: "~BG"
- board text removed: "~BGACK"
- board text removed: "~BR"
- board text removed: "~DTACK"
- board text removed: "~DTACK~ GROUNDED!!"
- board text removed: "~HALT"
- board text removed: "~IPL0"
- board text removed: "~IPL1"
- board text removed: "~IPL2"
- board text removed: "~LDS"
- board text removed: "~RDL"
- board text removed: "~RDU"
- board text removed: "~RESET"
- board text removed: "~RST"
- board text removed: "~SS"
- board text removed: "~UDS"
- board text removed: "~VMA"
- board text removed: "~VPA"
- board text removed: "~WRL"
- board text removed: "~WRU"

Commit message: Clean KiCad migration artifacts
Routing:
- net (no net): track 39.2 -> 0.00 mm
- net /~{RDU}: vias 4 -> 3
Other:
- board text removed: "rev 1 . june 24 2020 . matt sarnoff . msarnoff.org"
