File: project-5/68000sbc.kicad_pcb (KiCad board)
At the start: 2 copper layers, 127 x 90.8 mm, 49 parts, among them J1 USB_B, J2 5V FTDI SERIAL, J3 RTC (SparkFun BOB-10160), J4 CFCARD/IDE, J5 EXPANSION (F.Cu), J6 EXPANSION (B.Cu), SW1 RESET, SW2 BTN1, U1 74HC139, U2 74HC14, U3 TMP68HC000P-12, U4 AS6C4008-55PCN, U5 28C256, U6 AS6C4008-55PCN, U7 28C256, U8 TL16C550, X1 12MHz, X2 12MHz

Commit message: Amend fiver
Other:
- board text added: "68k magic"
- board text added: "cartheur"
- board text removed: "68k nano"
- board text removed: "rev 1 . june 24 2020 . matt sarnoff . msarnoff.org"
- board text removed: "single board computer"
Changed lines of the file:
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@@
-(kicad_pcb (version 20171130) (host pcbnew "(5.1.5-0-10_14)")
+(kicad_pcb (version 20171130) (host pcbnew "(5.1.5)-3")
   (general
     (thickness 1.6)
-    (drawings 172)
+    (drawings 171)
     (tracks 1753)
     (zones 0)
@@
     (solder_mask_min_width 0.25)
     (aux_axis_origin 0 0)
-    (visible_elements FFFFFF7F)
+    (visible_elements 7FFFFFFF)
     (pcbplotparams
       (layerselection 0x010f0_ffffffff)
@@
       (drillshape 0)
       (scaleselection 1)
-      (outputdirectory "gerbers/"))
+      (outputdirectory "../project-10-recovery/gerbers/"))
   )
   (net 0 "")
@@
   (gr_line (start 151.765 43.18) (end 153.035 43.18) (layer F.SilkS) (width 0.12))
   (gr_line (start 152.4 41.91) (end 151.765 43.18) (layer F.SilkS) (width 0.12))
-  (gr_text "rev 1 . june 24 2020 . matt sarnoff . msarnoff.org" (at 68.58 128.27) (layer F.SilkS)
+  (gr_text cartheur (at 68.58 128.27) (layer F.SilkS)
     (effects (font (size 1 1) (thickness 0.15) italic))
   )
-  (gr_text "single board computer" (at 57.785 42.926) (layer F.SilkS)
-    (effects (font (size 1.016 1.016) (thickness 0.254) italic))
-  )
-  (gr_text "68k nano" (at 56.261 40.894) (layer F.SilkS)
+  (gr_text "68k magic" (at 56.261 40.894) (layer F.SilkS)
     (effects (font (size 2.032 2.032) (thickness 0.508) italic))
   )
